Commit message: first link working finally :)))

File: urdf/robot.urdf (robot description, URDF)
Before this commit: robot robot_arm, 1 links, 0 joints
Links:
- link base_link: geometry collision cylinder length=0.3 radius=0.05; visual mesh filename=package://robot_arm_control_pkg/meshes/base.stl scale=0.001 0.001 0.001

Commit message: added first xacro in urdf

File: urdf/robot.urdf (robot description, URDF)
Before this commit: robot robot, 1 links, 0 joints
Links:
- link base_link: geometry collision cylinder length=${base_height} radius=${base_radius}; visual mesh filename=package://robot_arm_control_pkg/meshes/base.stl scale=0.001 0.001 0.001

Commit message: current links are now in urdf file

File: urdf/robot.urdf (robot description, URDF)
Before this commit: robot robot, 1 links, 0 joints
Links:
- added link shoulder_link; collision mesh filename=${mesh_path}/shoulder_link_collision.stl scale=0.001 0.001 0.001; visual mesh filename=${mesh_path}/shoulder_link.stl scale=0.001 0.001 0.001
- added link upper_arm_link; collision mesh filename=${mesh_path}/upper_arm_collision.stl scale=0.001 0.001 0.001; visual mesh filename=${mesh_path}/upper_arm.stl scale=0.001 0.001 0.001
- link base_link: geometry collision cylinder length=${base_height} radius=${base_radius}; visual mesh filename=${mesh_path}/base.stl scale=0.001 0.001 0.001
Joints:
- added joint base_joint: type revolute, parent base_link, child shoulder_link, origin xyz=0 0 ${base_height-0.0042} rpy=0 0 0, axis 0 0 1 , limit lower=${-PI} upper=${PI} effort=0.1 velocity=0.1
- added joint shoulder_joint: type revolute, parent shoulder_link, child upper_arm_link, origin xyz=-0.0008 0 0.0458 rpy=0 0 0, axis 0 0 1 , limit lower=${-PI} upper=${PI} effort=0.1 velocity=0.1

Commit message: URDF setup etc

File: urdf/robot.urdf (robot description, URDF)
Before this commit: robot robot, 3 links, 2 joints
Joints:
- joint base_joint: limit lower=${-PI} upper=${PI} effort=0.1 velocity=0.1 -> lower=${-PI/2} upper=${PI/2} effort=0.1 velocity=0.1
- joint shoulder_joint: axis 0 0 1  -> 1 0 0 ; limit lower=${-PI} upper=${PI} effort=0.1 velocity=0.1 -> lower=${-PI/2} upper=${PI/2} effort=0.1 velocity=0.1; origin xyz=-0.0008 0 0.0458 rpy=0 0 0 -> xyz=-0.0008 0 0.0458 rpy=${5.5*PI/180} 0 0
